File: left-keyboard-kicad-project/keyboard.kicad_sch (KiCad schematic)
At the start: 78 parts, among them U1 Arduino_Pro_Micro, U2 TRRS

Commit message: added hotswap sockets
Parts:
- K_1, K_2, K_3, K_4, K_5, K_6, K_A1, K_B1, K_C1, K_D1, K_E1, K_ESC1, K_F1, K_F2, K_F3, K_F4, K_F5, K_F6, K_G1, K_Q1, K_R1, K_S1, K_T1, K_V1, K_W1, K_X1, K_Y1, K_Z1, K_`1: footprint MX_ALPS_Hybrid:MXOnly-1U-NoLED -> MX_Alps_Hybrid_3:MXOnly-1U-Hotswap
- K_ALT1, K_CTRL1, K_FN1, K_WIN1: footprint MX_ALPS_Hybrid:MXOnly-1.25U-NoLED -> MX_Alps_Hybrid_3:MXOnly-1.25U-Hotswap
- K_CAPS1: footprint MX_ALPS_Hybrid:MXOnly-1.75U-NoLED -> MX_Alps_Hybrid_3:MXOnly-1.75U-Hotswap
- K_SHIFT1, K_SPACE1: footprint MX_ALPS_Hybrid:MXOnly-2.25U-NoLED -> MX_Alps_Hybrid_3:MXOnly-2.25U-Hotswap
- K_TAB1: footprint MX_ALPS_Hybrid:MXOnly-1.5U-NoLED -> MX_Alps_Hybrid_3:MXOnly-1.5U-Hotswap
