File: right-keyboard-kicad-project/keyboard.kicad_pcb (KiCad board)
At the start: 2 copper layers, 222.5 x 157.3 mm, 119 parts, among them SW1 SW_PUSH, U1 ATMEGA32U4, X1 XTAL_GND

Commit message: started right keyboard Kicad project
Parts:
- removed C1, C2, C3, C4, C5, C6, C7: 22pF, Capacitor_SMD:C_0805_2012Metric_Pad1.15x1.40mm_HandSolder
- removed the D_0 at (113.0, 33.8)
- removed the D_6 at (36.8, 33.8)
- removed the D_7 at (55.9, 33.8)
- removed the D_8 at (74.9, 33.8)
- removed the D_9 at (94.0, 33.8)
- removed the D_F10 at (113.0, 10.0)
- removed the D_F11 at (132.1, 10.0)
- removed the D_F12 at (151.1, 10.0)
- removed the D_F6 at (36.8, 10.0)
- removed the D_F7 at (55.9, 10.0)
- removed the D_F8 at (74.9, 10.0)
- removed the D_F9 at (94.0, 10.0)
- removed the K_0 at (103.0, 33.3)
- removed the K_6 at (26.8, 33.3)
- removed the K_7 at (45.8, 33.3)
- removed the K_8 at (64.9, 33.3)
- removed the K_9 at (83.9, 33.3)
- removed the K_F10 at (103.0, 9.53)
- removed the K_F11 at (122.0, 9.53)
- removed the K_F12 at (141.1, 9.53)
- removed the K_F6 at (26.8, 9.53)
- removed the K_F7 at (45.8, 9.53)
- removed the K_F8 at (64.9, 9.53)
- removed the K_F9 at (83.9, 9.53)
- removed R1, R2: 10k, Resistor_SMD:R_0805_2012Metric_Pad1.15x1.40mm_HandSolder
- removed R3, R4: 22, Resistor_SMD:R_0805_2012Metric_Pad1.15x1.40mm_HandSolder
- removed SW1: SW_PUSH, Button_Switch_SMD:SW_SPST_TL3342
- removed USB1: Molex-0548190589, keyboard_parts:Molex-0548190589-Assembly
- removed X1: XTAL_GND, Crystal:Crystal_SMD_5032-4Pin_5.0x3.2mm
- added D_0: D, keyboard_parts:D_SOD123_axial, F.Cu at (443.4, 37.7)
- added D_0: D, keyboard_parts:D_SOD123_axial, F.Cu at (168.8, 68.0)
- added D_6: D, keyboard_parts:D_SOD123_axial, F.Cu at (443.4, 41.3)
- added D_6: D, keyboard_parts:D_SOD123_axial, F.Cu at (92.6, 68.0)
- added D_7: D, keyboard_parts:D_SOD123_axial, F.Cu at (111.7, 68.0)
- added D_7: D, keyboard_parts:D_SOD123_axial, F.Cu at (443.4, 44.9)
- added D_8: D, keyboard_parts:D_SOD123_axial, F.Cu at (130.7, 68.0)
- added D_8: D, keyboard_parts:D_SOD123_axial, F.Cu at (443.4, 48.5)
- added D_9: D, keyboard_parts:D_SOD123_axial, F.Cu at (149.8, 68.0)
- added D_9: D, keyboard_parts:D_SOD123_axial, F.Cu at (443.4, 52.1)
- added D_ALT1: D, keyboard_parts:D_SOD123_axial, F.Cu at (443.4, 55.7)
- added D_B1: D, keyboard_parts:D_SOD123_axial, F.Cu at (443.4, 59.3)
- added D_BACKSPACE1: D, keyboard_parts:D_SOD123_axial, F.Cu at (443.4, 62.9)
- added D_BSLSH1: D, keyboard_parts:D_SOD123_axial, F.Cu at (443.4, 66.5)
- added D_CBRAC1: D, keyboard_parts:D_SOD123_axial, F.Cu at (443.4, 70.1)
- added D_COMMA1: D, keyboard_parts:D_SOD123_axial, F.Cu at (443.4, 73.7)
- added D_CTRL1: D, keyboard_parts:D_SOD123_axial, F.Cu at (443.4, 77.3)
- added D_DELETE1: D, keyboard_parts:D_SOD123_axial, F.Cu at (443.4, 80.9)
- added D_DOT1: D, keyboard_parts:D_SOD123_axial, F.Cu at (443.4, 84.5)
- added D_DOWN1: D, keyboard_parts:D_SOD123_axial, F.Cu at (453.8, 37.7)
- added D_END1: D, keyboard_parts:D_SOD123_axial, F.Cu at (453.8, 41.3)
- added D_ENTER1: D, keyboard_parts:D_SOD123_axial, F.Cu at (453.8, 44.9)
- added D_EQUAL1: D, keyboard_parts:D_SOD123_axial, F.Cu at (453.8, 48.5)
- added D_F10: D, keyboard_parts:D_SOD123_axial, F.Cu at (453.8, 66.5)
- added D_F10: D, keyboard_parts:D_SOD123_axial, F.Cu at (168.8, 44.1)
- added D_F11: D, keyboard_parts:D_SOD123_axial, F.Cu at (187.9, 44.1)
- added D_F11: D, keyboard_parts:D_SOD123_axial, F.Cu at (453.8, 70.1)
- added D_F12: D, keyboard_parts:D_SOD123_axial, F.Cu at (453.8, 73.7)
- added D_F12: D, keyboard_parts:D_SOD123_axial, F.Cu at (206.9, 44.1)
- added D_F6: D, keyboard_parts:D_SOD123_axial, F.Cu at (92.6, 44.1)
- added D_F6: D, keyboard_parts:D_SOD123_axial, F.Cu at (453.8, 52.1)
- added D_F7: D, keyboard_parts:D_SOD123_axial, F.Cu at (111.7, 44.1)
- added D_F7: D, keyboard_parts:D_SOD123_axial, F.Cu at (453.8, 55.7)
- added D_F8: D, keyboard_parts:D_SOD123_axial, F.Cu at (130.7, 44.1)
- added D_F8: D, keyboard_parts:D_SOD123_axial, F.Cu at (453.8, 59.3)
- added D_F9: D, keyboard_parts:D_SOD123_axial, F.Cu at (453.8, 62.9)
- added D_F9: D, keyboard_parts:D_SOD123_axial, F.Cu at (149.8, 44.1)
- added D_FN1: D, keyboard_parts:D_SOD123_axial, F.Cu at (453.8, 77.3)
- added D_H1: D, keyboard_parts:D_SOD123_axial, F.Cu at (453.8, 80.9)
- added D_HOME1: D, keyboard_parts:D_SOD123_axial, F.Cu at (453.8, 84.5)
- added D_I1: D, keyboard_parts:D_SOD123_axial, F.Cu at (464.2, 37.7)
- added D_J1: D, keyboard_parts:D_SOD123_axial, F.Cu at (464.2, 41.3)
- added D_K1: D, keyboard_parts:D_SOD123_axial, F.Cu at (464.2, 44.9)
- added D_L1: D, keyboard_parts:D_SOD123_axial, F.Cu at (464.2, 48.5)
- added D_LEFT1: D, keyboard_parts:D_SOD123_axial, F.Cu at (464.2, 52.1)
- added D_M1: D, keyboard_parts:D_SOD123_axial, F.Cu at (464.2, 55.7)
- added D_MINUS1: D, keyboard_parts:D_SOD123_axial, F.Cu at (464.2, 59.3)
- added D_N1: D, keyboard_parts:D_SOD123_axial, F.Cu at (464.2, 62.9)
- added D_O1: D, keyboard_parts:D_SOD123_axial, F.Cu at (464.2, 66.5)
- added D_OBRAC1: D, keyboard_parts:D_SOD123_axial, F.Cu at (464.2, 70.1)
- added D_P1: D, keyboard_parts:D_SOD123_axial, F.Cu at (464.2, 73.7)
- added D_PGDN1: D, keyboard_parts:D_SOD123_axial, F.Cu at (464.2, 77.3)
- added D_PGUP1: D, keyboard_parts:D_SOD123_axial, F.Cu at (464.2, 80.9)
- added D_PRTSC1: D, keyboard_parts:D_SOD123_axial, F.Cu at (464.2, 84.5)
- added D_QUOTE1: D, keyboard_parts:D_SOD123_axial, F.Cu at (474.6, 37.7)
- added D_RIGHT1: D, keyboard_parts:D_SOD123_axial, F.Cu at (474.6, 41.3)
- added D_SEMIC1: D, keyboard_parts:D_SOD123_axial, F.Cu at (474.6, 44.9)
- added D_SHIFT1: D, keyboard_parts:D_SOD123_axial, F.Cu at (474.6, 48.5)
- added D_SLASH1: D, keyboard_parts:D_SOD123_axial, F.Cu at (474.6, 52.1)
- added D_SPACE1: D, keyboard_parts:D_SOD123_axial, F.Cu at (474.6, 55.7)
- added D_U1: D, keyboard_parts:D_SOD123_axial, F.Cu at (474.6, 59.3)
- added D_UP1: D, keyboard_parts:D_SOD123_axial, F.Cu at (474.6, 62.9)
- added D_WIN1: D, keyboard_parts:D_SOD123_axial, F.Cu at (474.6, 66.5)
- added D_Y1: D, keyboard_parts:D_SOD123_axial, F.Cu at (474.6, 70.1)
- added K_0: KEYSW, MX_Alps_Hybrid:MX-1U-NoLED, F.Cu at (158.8, 67.5)
- added K_0: KEYSW, MX_Alps_Hybrid_3:MXOnly-1U-Hotswap, F.Cu at (327.1, 46.0)
- added K_6: KEYSW, MX_Alps_Hybrid_3:MXOnly-1U-Hotswap, F.Cu at (327.1, 66.2)
- added K_6: KEYSW, MX_Alps_Hybrid:MX-1U-NoLED, F.Cu at (82.6, 67.5)
- added K_7: KEYSW, MX_Alps_Hybrid_3:MXOnly-1U-Hotswap, F.Cu at (327.1, 86.4)
- added K_7: KEYSW, MX_Alps_Hybrid:MX-1U-NoLED, F.Cu at (101.6, 67.5)
- added K_8: KEYSW, MX_Alps_Hybrid:MX-1U-NoLED, F.Cu at (120.7, 67.5)
- added K_8: KEYSW, MX_Alps_Hybrid_3:MXOnly-1U-Hotswap, F.Cu at (327.1, 106.6)
- added K_9: KEYSW, MX_Alps_Hybrid_3:MXOnly-1U-Hotswap, F.Cu at (327.1, 126.8)
- added K_9: KEYSW, MX_Alps_Hybrid:MX-1U-NoLED, F.Cu at (139.7, 67.5)
- added K_ALT1: KEYSW, MX_Alps_Hybrid_3:MXOnly-1U-Hotswap, F.Cu at (327.1, 147.0)
- added K_B1: KEYSW, MX_Alps_Hybrid_3:MXOnly-1U-Hotswap, F.Cu at (327.1, 167.2)
- added K_BACKSPACE1: KEYSW, MX_Alps_Hybrid_3:MXOnly-2U-Hotswap, F.Cu at (457.8, 138.1)
- added K_BSLSH1: KEYSW, MX_Alps_Hybrid_3:MXOnly-1.5U-Hotswap, F.Cu at (472.0, 179.1)
- added K_CBRAC1: KEYSW, MX_Alps_Hybrid_3:MXOnly-1U-Hotswap, F.Cu at (327.1, 187.4)
- added K_COMMA1: KEYSW, MX_Alps_Hybrid_3:MXOnly-1U-Hotswap, F.Cu at (347.3, 46.0)
- added K_CTRL1: KEYSW, MX_Alps_Hybrid_3:MXOnly-1U-Hotswap, F.Cu at (347.3, 66.2)
- added K_DELETE1: KEYSW, MX_Alps_Hybrid_3:MXOnly-1U-Hotswap, F.Cu at (347.3, 86.4)
- added K_DOT1: KEYSW, MX_Alps_Hybrid_3:MXOnly-1U-Hotswap, F.Cu at (347.3, 106.6)
- added K_DOWN1: KEYSW, MX_Alps_Hybrid_3:MXOnly-1U-Hotswap, F.Cu at (347.3, 126.8)
- added K_END1: KEYSW, MX_Alps_Hybrid_3:MXOnly-1U-Hotswap, F.Cu at (347.3, 147.0)
- added K_ENTER1: KEYSW, MX_Alps_Hybrid_3:MXOnly-2.25U-Hotswap, F.Cu at (460.2, 96.4)
- added K_EQUAL1: KEYSW, MX_Alps_Hybrid_3:MXOnly-1U-Hotswap, F.Cu at (347.3, 167.2)
- added K_F10: KEYSW, MX_Alps_Hybrid_3:MXOnly-1U-Hotswap, F.Cu at (367.5, 106.6)
- added K_F10: KEYSW, MX_Alps_Hybrid:MX-1U-NoLED, F.Cu at (158.8, 43.6)
- added K_F11: KEYSW, MX_Alps_Hybrid_3:MXOnly-1U-Hotswap, F.Cu at (367.5, 126.8)
- added K_F11: KEYSW, MX_Alps_Hybrid:MX-1U-NoLED, F.Cu at (177.8, 43.6)
- added K_F12: KEYSW, MX_Alps_Hybrid:MX-1U-NoLED, F.Cu at (196.9, 43.6)
- added K_F12: KEYSW, MX_Alps_Hybrid_3:MXOnly-1U-Hotswap, F.Cu at (367.5, 147.0)
- added K_F6: KEYSW, MX_Alps_Hybrid_3:MXOnly-1U-Hotswap, F.Cu at (347.3, 187.4)
- added K_F6: KEYSW, MX_Alps_Hybrid:MX-1U-NoLED, F.Cu at (82.6, 43.6)
- added K_F7: KEYSW, MX_Alps_Hybrid_3:MXOnly-1U-Hotswap, F.Cu at (367.5, 46.0)
- added K_F7: KEYSW, MX_Alps_Hybrid:MX-1U-NoLED, F.Cu at (101.6, 43.6)
- added K_F8: KEYSW, MX_Alps_Hybrid:MX-1U-NoLED, F.Cu at (120.7, 43.6)
- added K_F8: KEYSW, MX_Alps_Hybrid_3:MXOnly-1U-Hotswap, F.Cu at (367.5, 66.2)
- added K_F9: KEYSW, MX_Alps_Hybrid:MX-1U-NoLED, F.Cu at (139.7, 43.6)
- added K_F9: KEYSW, MX_Alps_Hybrid_3:MXOnly-1U-Hotswap, F.Cu at (367.5, 86.4)
- added K_FN1: KEYSW, MX_Alps_Hybrid_3:MXOnly-1U-Hotswap, F.Cu at (367.5, 167.2)
- added K_H1: KEYSW, MX_Alps_Hybrid_3:MXOnly-1U-Hotswap, F.Cu at (367.5, 187.4)
- added K_HOME1: KEYSW, MX_Alps_Hybrid_3:MXOnly-1U-Hotswap, F.Cu at (387.7, 46.0)
- added K_I1: KEYSW, MX_Alps_Hybrid_3:MXOnly-1U-Hotswap, F.Cu at (387.7, 66.2)
- added K_J1: KEYSW, MX_Alps_Hybrid_3:MXOnly-1U-Hotswap, F.Cu at (387.7, 86.4)
- added K_K1: KEYSW, MX_Alps_Hybrid_3:MXOnly-1U-Hotswap, F.Cu at (387.7, 106.6)
- added K_L1: KEYSW, MX_Alps_Hybrid_3:MXOnly-1U-Hotswap, F.Cu at (387.7, 126.8)
- added K_LEFT1: KEYSW, MX_Alps_Hybrid_3:MXOnly-1U-Hotswap, F.Cu at (387.7, 147.0)
- added K_M1: KEYSW, MX_Alps_Hybrid_3:MXOnly-1U-Hotswap, F.Cu at (387.7, 167.2)
- added K_MINUS1: KEYSW, MX_Alps_Hybrid_3:MXOnly-1U-Hotswap, F.Cu at (387.7, 187.4)
- added K_N1: KEYSW, MX_Alps_Hybrid_3:MXOnly-1U-Hotswap, F.Cu at (407.9, 46.0)
- added K_O1: KEYSW, MX_Alps_Hybrid_3:MXOnly-1U-Hotswap, F.Cu at (407.9, 66.2)
- added K_OBRAC1: KEYSW, MX_Alps_Hybrid_3:MXOnly-1U-Hotswap, F.Cu at (407.9, 86.4)
- added K_P1: KEYSW, MX_Alps_Hybrid_3:MXOnly-1U-Hotswap, F.Cu at (407.9, 106.6)
- added K_PGDN1: KEYSW, MX_Alps_Hybrid_3:MXOnly-1U-Hotswap, F.Cu at (407.9, 126.8)
- added K_PGUP1: KEYSW, MX_Alps_Hybrid_3:MXOnly-1U-Hotswap, F.Cu at (407.9, 147.0)
- added K_PRTSC1: KEYSW, MX_Alps_Hybrid_3:MXOnly-1U-Hotswap, F.Cu at (407.9, 167.2)
- added K_QUOTE1: KEYSW, MX_Alps_Hybrid_3:MXOnly-1U-Hotswap, F.Cu at (407.9, 187.4)
- added K_RIGHT1: KEYSW, MX_Alps_Hybrid_3:MXOnly-1U-Hotswap, F.Cu at (428.1, 46.0)
- added K_SEMIC1: KEYSW, MX_Alps_Hybrid_3:MXOnly-1U-Hotswap, F.Cu at (428.1, 66.2)
- added K_SHIFT1: KEYSW, MX_Alps_Hybrid_3:MXOnly-1.75U-Hotswap, F.Cu at (474.4, 158.9)
- added K_SLASH1: KEYSW, MX_Alps_Hybrid_3:MXOnly-1U-Hotswap, F.Cu at (428.1, 86.4)
- added K_SPACE1: KEYSW, MX_Alps_Hybrid_3:MXOnly-2.25U-Hotswap, F.Cu at (460.2, 117.2)
- added K_U1: KEYSW, MX_Alps_Hybrid_3:MXOnly-1U-Hotswap, F.Cu at (428.1, 106.6)
- added K_UP1: KEYSW, MX_Alps_Hybrid_3:MXOnly-1U-Hotswap, F.Cu at (428.1, 126.8)
- added K_WIN1: KEYSW, MX_Alps_Hybrid_3:MXOnly-1U-Hotswap, F.Cu at (428.1, 147.0)
- added K_Y1: KEYSW, MX_Alps_Hybrid_3:MXOnly-1U-Hotswap, F.Cu at (428.1, 167.2)
- added U2: Arduino_Pro_Micro, ScottoKeebs_MCU:Arduino_Pro_Micro, F.Cu at (447.6, 168.7)
- U1: value ATMEGA32U4 -> TRRS; footprint Package_QFP:TQFP-44_10x10mm_P0.8mm -> ScottoKeebs_Components:TRRS_PJ-320A; moved to F.Cu
- moved U1 279.3 mm to (481.0, 130.6)
- moved D_ALT 65.4 mm to (149.8, 144.2)
- moved D_DOWN 65.4 mm to (249.8, 144.2)
- moved D_FN 65.4 mm to (187.9, 144.2)
- moved K_ALT 65.4 mm to (139.7, 143.7)
- moved K_CTRL 65.4 mm to (196.9, 143.7)
- moved K_DOWN 65.4 mm to (239.8, 143.7)
- moved K_FN 65.4 mm to (177.8, 143.7)
- moved K_LEFT 65.4 mm to (220.7, 143.7)
- moved K_RIGHT 65.4 mm to (258.8, 143.7)
- moved D_BACKSPACE 65.4 mm to (245.0, 68.0)
- moved D_BSLSH 65.4 mm to (245.0, 87.0)
- moved D_CBRAC 65.4 mm to (197.4, 87.0)
- moved D_COMMA 65.4 mm to (154.5, 125.1)
- moved D_DOT 65.4 mm to (173.6, 125.1)
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Connections:
- U1 pad 1: Net-(U1-Pad1) -> unconnected-(U1-SLEEVE-Pad1)
- U1 pad 2: VCC -> unconnected-(U1-TIP-Pad2)
- U1 pad 3: Net-(R3-Pad1) -> unconnected-(U1-RING1-Pad3)
- U1 pad 4: Net-(R4-Pad1) -> unconnected-(U1-RING2-Pad4)
Routing:
- removed copper zone on B.Cu, net GND
- removed copper zone on F.Cu, net VCC
Other:
- board outline removed
- net class Default removed
- board text removed: "PCB Builder by MisterKeebs - mrkeebs.com"

Commit message: Redid right keyboard firmware wiring and started right keyboard Kicad project
Parts:
- removed the D_0 at (443.4, 37.7)
- removed the D_0 at (168.8, 68.0)
- removed the D_6 at (443.4, 41.3)
- removed the D_6 at (92.6, 68.0)
- removed the D_7 at (111.7, 68.0)
- removed the D_7 at (443.4, 44.9)
- removed the D_8 at (130.7, 68.0)
- removed the D_8 at (443.4, 48.5)
- removed the D_9 at (149.8, 68.0)
- removed the D_9 at (443.4, 52.1)
- removed the D_F10 at (453.8, 66.5)
- removed the D_F10 at (168.8, 44.1)
- removed the D_F11 at (187.9, 44.1)
- removed the D_F11 at (453.8, 70.1)
- removed the D_F12 at (453.8, 73.7)
- removed the D_F12 at (206.9, 44.1)
- removed the D_F6 at (92.6, 44.1)
- removed the D_F6 at (453.8, 52.1)
- removed the D_F7 at (111.7, 44.1)
- removed the D_F7 at (453.8, 55.7)
- removed the D_F8 at (130.7, 44.1)
- removed the D_F8 at (453.8, 59.3)
- removed the D_F9 at (453.8, 62.9)
- removed the D_F9 at (149.8, 44.1)
- removed the K_0 at (158.8, 67.5)
- removed the K_0 at (327.1, 46.0)
- removed the K_6 at (327.1, 66.2)
- removed the K_6 at (82.6, 67.5)
- removed the K_7 at (327.1, 86.4)
- removed the K_7 at (101.6, 67.5)
- removed the K_8 at (120.7, 67.5)
- removed the K_8 at (327.1, 106.6)
- removed the K_9 at (327.1, 126.8)
- removed the K_9 at (139.7, 67.5)
- removed the K_F10 at (367.5, 106.6)
- removed the K_F10 at (158.8, 43.6)
- removed the K_F11 at (367.5, 126.8)
- removed the K_F11 at (177.8, 43.6)
- removed the K_F12 at (196.9, 43.6)
- removed the K_F12 at (367.5, 147.0)
- removed the K_F6 at (347.3, 187.4)
- removed the K_F6 at (82.6, 43.6)
- removed the K_F7 at (367.5, 46.0)
- removed the K_F7 at (101.6, 43.6)
- removed the K_F8 at (120.7, 43.6)
- removed the K_F8 at (367.5, 66.2)
- removed the K_F9 at (139.7, 43.6)
- removed the K_F9 at (367.5, 86.4)
- added D_0: D, keyboard_parts:D_SOD123_axial, F.Cu at (166.9, 82.1)
- added D_0: D, keyboard_parts:D_SOD123_axial, F.Cu at (431.5, 39.8)
- added D_6: D, keyboard_parts:D_SOD123_axial, F.Cu at (90.8, 82.1)
- added D_6: D, keyboard_parts:D_SOD123_axial, F.Cu at (431.5, 43.4)
- added D_7: D, keyboard_parts:D_SOD123_axial, F.Cu at (109.8, 82.1)
- added D_7: D, keyboard_parts:D_SOD123_axial, F.Cu at (431.5, 47.0)
- added D_8: D, keyboard_parts:D_SOD123_axial, F.Cu at (431.5, 50.6)
- added D_8: D, keyboard_parts:D_SOD123_axial, F.Cu at (128.8, 82.1)
- added D_9: D, keyboard_parts:D_SOD123_axial, F.Cu at (431.5, 54.2)
- added D_9: D, keyboard_parts:D_SOD123_axial, F.Cu at (147.9, 82.1)
- added D_F10: D, keyboard_parts:D_SOD123_axial, F.Cu at (441.9, 68.6)
- added D_F10: D, keyboard_parts:D_SOD123_axial, F.Cu at (166.9, 58.2)
- added D_F11: D, keyboard_parts:D_SOD123_axial, F.Cu at (186.0, 58.2)
- added D_F11: D, keyboard_parts:D_SOD123_axial, F.Cu at (441.9, 72.2)
- added D_F12: D, keyboard_parts:D_SOD123_axial, F.Cu at (441.9, 75.8)
- added D_F12: D, keyboard_parts:D_SOD123_axial, F.Cu at (205.1, 58.2)
- added D_F6: D, keyboard_parts:D_SOD123_axial, F.Cu at (90.8, 58.2)
- added D_F6: D, keyboard_parts:D_SOD123_axial, F.Cu at (441.9, 54.2)
- added D_F7: D, keyboard_parts:D_SOD123_axial, F.Cu at (441.9, 57.8)
- added D_F7: D, keyboard_parts:D_SOD123_axial, F.Cu at (109.8, 58.2)
- added D_F8: D, keyboard_parts:D_SOD123_axial, F.Cu at (128.8, 58.2)
- added D_F8: D, keyboard_parts:D_SOD123_axial, F.Cu at (441.9, 61.4)
- added D_F9: D, keyboard_parts:D_SOD123_axial, F.Cu at (147.9, 58.2)
- added D_F9: D, keyboard_parts:D_SOD123_axial, F.Cu at (441.9, 65.0)
- added K_0: KEYSW, MX_Alps_Hybrid:MX-1U-NoLED, F.Cu at (156.9, 81.6)
- added K_0: KEYSW, MX_Alps_Hybrid_3:MXOnly-1U-Hotswap, F.Cu at (315.2, 48.1)
- added K_6: KEYSW, MX_Alps_Hybrid_3:MXOnly-1U-Hotswap, F.Cu at (315.2, 68.3)
- added K_6: KEYSW, MX_Alps_Hybrid:MX-1U-NoLED, F.Cu at (80.7, 81.6)
- added K_7: KEYSW, MX_Alps_Hybrid:MX-1U-NoLED, F.Cu at (99.8, 81.6)
- added K_7: KEYSW, MX_Alps_Hybrid_3:MXOnly-1U-Hotswap, F.Cu at (315.2, 88.5)
- added K_8: KEYSW, MX_Alps_Hybrid_3:MXOnly-1U-Hotswap, F.Cu at (315.2, 108.7)
- added K_8: KEYSW, MX_Alps_Hybrid:MX-1U-NoLED, F.Cu at (118.8, 81.6)
- added K_9: KEYSW, MX_Alps_Hybrid:MX-1U-NoLED, F.Cu at (137.9, 81.6)
- added K_9: KEYSW, MX_Alps_Hybrid_3:MXOnly-1U-Hotswap, F.Cu at (315.2, 128.9)
- added K_F10: KEYSW, MX_Alps_Hybrid_3:MXOnly-1U-Hotswap, F.Cu at (355.6, 108.7)
- added K_F10: KEYSW, MX_Alps_Hybrid:MX-1U-NoLED, F.Cu at (156.9, 57.7)
- added K_F11: KEYSW, MX_Alps_Hybrid:MX-1U-NoLED, F.Cu at (176.0, 57.7)
- added K_F11: KEYSW, MX_Alps_Hybrid_3:MXOnly-1U-Hotswap, F.Cu at (355.6, 128.9)
- added K_F12: KEYSW, MX_Alps_Hybrid_3:MXOnly-1U-Hotswap, F.Cu at (355.6, 149.1)
- added K_F12: KEYSW, MX_Alps_Hybrid:MX-1U-NoLED, F.Cu at (195.0, 57.7)
- added K_F6: KEYSW, MX_Alps_Hybrid_3:MXOnly-1U-Hotswap, F.Cu at (335.4, 189.5)
- added K_F6: KEYSW, MX_Alps_Hybrid:MX-1U-NoLED, F.Cu at (80.7, 57.7)
- added K_F7: KEYSW, MX_Alps_Hybrid_3:MXOnly-1U-Hotswap, F.Cu at (355.6, 48.1)
- added K_F7: KEYSW, MX_Alps_Hybrid:MX-1U-NoLED, F.Cu at (99.8, 57.7)
- added K_F8: KEYSW, MX_Alps_Hybrid:MX-1U-NoLED, F.Cu at (118.8, 57.7)
- added K_F8: KEYSW, MX_Alps_Hybrid_3:MXOnly-1U-Hotswap, F.Cu at (355.6, 68.3)
- added K_F9: KEYSW, MX_Alps_Hybrid_3:MXOnly-1U-Hotswap, F.Cu at (355.6, 88.5)
- added K_F9: KEYSW, MX_Alps_Hybrid:MX-1U-NoLED, F.Cu at (137.9, 57.7)
- U1: value TRRS -> Arduino_Pro_Micro; footprint ScottoKeebs_Components:TRRS_PJ-320A -> ScottoKeebs_MCU:Arduino_Pro_Micro
- U2: value Arduino_Pro_Micro -> TRRS; footprint ScottoKeebs_MCU:Arduino_Pro_Micro -> ScottoKeebs_Components:TRRS_PJ-320A
- moved U1 60.6 mm to (435.8, 170.8)
- moved U2 42.0 mm to (469.2, 132.7)
- moved D_SPACE 14.2 mm to (113.8, 158.9)
- moved K_SPACE 14.2 mm to (91.9, 158.4)
- moved D_PGDN 14.2 mm to (243.2, 58.2)
- moved D_PGUP 14.2 mm to (224.1, 58.2)
- moved D_PRTSC 14.2 mm to (267.0, 58.2)
- moved K_PGDN 14.2 mm to (233.1, 57.7)
- moved K_PGUP 14.2 mm to (214.1, 57.7)
- moved K_PRTSC 14.2 mm to (256.9, 57.7)
- moved D_ALT 14.2 mm to (147.9, 158.3)
- moved D_B 14.2 mm to (95.5, 139.2)
- moved D_BACKSPACE 14.2 mm to (243.2, 82.1)
- moved D_BSLSH 14.2 mm to (243.2, 101.1)
- moved D_CBRAC 14.2 mm to (195.5, 101.1)
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Connections:
- D_DELETE pad 1: /row1 -> /row2
- D_DELETE1 pad 1: row1 -> row2
- D_END pad 1: /row3 -> /row4
- D_END1 pad 1: row3 -> row4
- D_HOME pad 1: /row2 -> /row3
- D_HOME1 pad 1: row2 -> row3
- D_PRTSC pad 1: /row0 -> /row1
- D_PRTSC1 pad 1: row0 -> row1
- K_ALT pad 1: /col3 -> /col1
- K_ALT1 pad 1: col3 -> col1
- K_BSLSH pad 1: /col8 -> /col7
- K_BSLSH1 pad 1: col8 -> col7
- K_CTRL pad 1: /col6 -> /col4
- K_CTRL1 pad 1: col6 -> col4
- K_DELETE pad 1: /col9 -> /col8
- K_DELETE1 pad 1: col9 -> col8
- K_DOWN pad 1: /col8 -> /col6
- K_DOWN1 pad 1: col8 -> col6
- K_END pad 1: /col9 -> /col8
- K_END1 pad 1: col9 -> col8
- K_ENTER pad 1: /col7 -> /col6
- K_ENTER1 pad 1: col7 -> col6
- K_FN pad 1: /col5 -> /col3
- K_FN1 pad 1: col5 -> col3
- K_HOME pad 1: /col9 -> /col8
- K_HOME1 pad 1: col9 -> col8
- K_LEFT pad 1: /col7 -> /col5
- K_LEFT1 pad 1: col7 -> col5
- K_PRTSC pad 1: /col9 -> /col8
- K_PRTSC1 pad 1: col9 -> col8
- K_RIGHT pad 1: /col9 -> /col7
- K_RIGHT1 pad 1: col9 -> col7
- K_UP pad 1: /col8 -> /col7
- K_UP1 pad 1: col8 -> col7
- K_WIN pad 1: /col4 -> /col2
- K_WIN1 pad 1: col4 -> col2
- U1 pad 1: unconnected-(U1-SLEEVE-Pad1) -> Net-(U1-TX0/PD3)
- U1 pad 2: unconnected-(U1-TIP-Pad2) -> Net-(U1-RX1/PD2)
- U1 pad 3: unconnected-(U1-RING1-Pad3) -> GND
- U1 pad 4: unconnected-(U1-RING2-Pad4) -> GND
- U2 pad 1: unconnected-(U2-TX0/PD3-Pad1) -> GND
- U2 pad 2: unconnected-(U2-RX1/PD2-Pad2) -> Net-(U1-VCC)
- U2 pad 3: unconnected-(U2-GND-Pad3) -> Net-(U1-RX1/PD2)
- U2 pad 4: unconnected-(U2-GND-Pad4) -> Net-(U1-TX0/PD3)

Commit message: Completed placing switches and some diodes for right side
Parts:
- removed the D_0 at (166.9, 82.1)
- removed the D_6 at (90.8, 82.1)
- removed the D_7 at (109.8, 82.1)
- removed the D_8 at (128.8, 82.1)
- removed the D_9 at (147.9, 82.1)
- removed D_ALT, D_B, D_BACKSPACE, D_BSLSH, D_CBRAC, D_COMMA, D_CTRL, D_DELETE, D_DOT, D_DOWN, D_END, D_ENTER, D_EQUAL, D_FN, D_H, D_HOME, D_I, D_J, D_K, D_L, D_LEFT, D_M, D_MINUS, D_N, D_O, D_OBRAC, D_P, D_PGDN, D_PGUP, D_PRTSC, D_QUOTE, D_RIGHT, D_SEMIC, D_SHIFT, D_SLASH, D_SPACE, D_U, D_UP, D_WIN, D_Y: D, keyboard_parts:D_SOD123_axial
- removed the D_F10 at (166.9, 58.2)
- removed the D_F11 at (186.0, 58.2)
- removed the D_F12 at (205.1, 58.2)
- removed the D_F6 at (90.8, 58.2)
- removed the D_F7 at (109.8, 58.2)
- removed the D_F8 at (128.8, 58.2)
- removed the D_F9 at (147.9, 58.2)
- removed the K_0 at (156.9, 81.6)
- removed the K_6 at (80.7, 81.6)
- removed the K_7 at (99.8, 81.6)
- removed the K_8 at (118.8, 81.6)
- removed the K_9 at (137.9, 81.6)
- removed K_ALT, K_B, K_CBRAC, K_COMMA, K_CTRL, K_DELETE, K_DOT, K_DOWN, K_END, K_EQUAL, K_FN, K_H, K_HOME, K_I, K_J, K_K, K_L, K_LEFT, K_M, K_MINUS, K_N, K_O, K_OBRAC, K_P, K_PGDN, K_PGUP, K_PRTSC, K_QUOTE, K_RIGHT, K_SEMIC, K_SLASH, K_U, K_UP, K_WIN, K_Y: KEYSW, MX_Alps_Hybrid:MX-1U-NoLED
- removed K_BACKSPACE: KEYSW, MX_Alps_Hybrid:MX-2U-NoLED
- removed K_BSLSH: KEYSW, MX_Alps_Hybrid:MX-1.5U-NoLED
- removed K_ENTER, K_SPACE: KEYSW, MX_Alps_Hybrid:MX-2.25U-NoLED
- removed the K_F10 at (156.9, 57.7)
- removed the K_F11 at (176.0, 57.7)
- removed the K_F12 at (195.0, 57.7)
- removed the K_F6 at (80.7, 57.7)
- removed the K_F7 at (99.8, 57.7)
- removed the K_F8 at (118.8, 57.7)
- removed the K_F9 at (137.9, 57.7)
- removed K_SHIFT: KEYSW, MX_Alps_Hybrid:MX-1.75U-NoLED
- D_F10, D_F11, D_F12, D_F6, D_F7, D_F8, D_F9, D_PGDN1, D_PGUP1, D_PRTSC1, K_SPACE1, U1, U2: moved to B.Cu
- moved U2 437.4 mm to (40.4, 46.2), turned to 180 degrees
- moved U1 416.0 mm to (28.6, 85.7), turned to 180 degrees
- moved K_SPACE1 379.1 mm to (72.9, 172.2), turned to -60 degrees
- moved D_F6 352.0 mm to (89.9, 57.7), turned to 90 degrees
- moved K_Y1 333.1 mm to (90.2, 100.6)
- moved D_F7 332.9 mm to (109.0, 57.7), turned to 90 degrees
- moved D_F8 313.9 mm to (128.1, 57.7), turned to 90 degrees
- moved K_U1 307.0 mm to (109.3, 100.6)
- moved K_N1 305.2 mm to (104.5, 138.7)
- moved D_F9 294.9 mm to (147.1, 57.7), turned to 90 degrees
- moved D_0 288.9 mm to (181.3, 184.4)
- moved D_6 288.9 mm to (181.3, 188.0)
- moved D_7 288.9 mm to (181.3, 191.6)
- moved D_8 288.9 mm to (181.3, 195.2)
- moved D_9 288.9 mm to (181.3, 198.8)
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
Commit message: Finished right side of keyboard
Parts:
- D_0, D_6, D_7, D_8, D_9, D_ALT1, D_B1, D_BACKSPACE1, D_BSLSH1, D_CBRAC1, D_COMMA1, D_CTRL1, D_DELETE1, D_DOT1, D_DOWN1, D_END1, D_ENTER1, D_EQUAL1, D_FN1, D_H1, D_HOME1, D_I1, D_J1, D_K1, D_L1, D_LEFT1, D_M1, D_MINUS1, D_N1, D_O1, D_OBRAC1, D_P1, D_QUOTE1, D_RIGHT1, D_SEMIC1, D_SHIFT1, D_SLASH1, D_SPACE1, D_U1, D_UP1, D_WIN1, D_Y1: moved to B.Cu
- K_SPACE1, U1, U2: moved to F.Cu
- moved D_BACKSPACE1 311.5 mm to (496.9, 78.7), turned to 90 degrees
- moved D_EQUAL1 292.0 mm to (459.5, 78.7), turned to 90 degrees
- moved U1 281.1 mm to (308.5, 60.2), turned to 0 degrees
- moved D_MINUS1 270.1 mm to (440.4, 78.7), turned to 90 degrees
- moved D_0 262.3 mm to (421.3, 78.6), turned to 90 degrees
- moved K_DELETE1 255.2 mm to (512.1, 78.7)
- moved K_END1 255.2 mm to (512.1, 116.8)
- moved K_HOME1 255.2 mm to (512.1, 97.8)
- moved K_PRTSC1 255.2 mm to (512.1, 54.9)
- moved K_RIGHT1 255.2 mm to (512.1, 154.9)
- moved D_F9 255.2 mm to (402.3, 54.9)
- moved D_PGDN1 255.2 mm to (497.5, 54.8)
- moved D_PGUP1 255.2 mm to (478.5, 54.8)
- moved K_6 255.2 mm to (335.9, 78.7)
- moved K_BACKSPACE1 255.2 mm to (478.8, 78.7)
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Routing:
- net row5: track 0.00 -> 304.9 mm, vias 0 -> 1
- net col8: track 0.00 -> 299.6 mm, vias 0 -> 4
- net col7: track 0.00 -> 284.3 mm, vias 0 -> 2
- net row4: track 0.00 -> 279.1 mm
- net col6: track 0.00 -> 271.5 mm, vias 0 -> 1
- net row3: track 0.00 -> 270.7 mm
- net col5: track 0.00 -> 250.7 mm, vias 0 -> 1
- net row2: track 0.00 -> 249.0 mm
- net row1: track 0.00 -> 240.3 mm
- net col4: track 0.00 -> 229.3 mm, vias 0 -> 3
- net col3: track 0.00 -> 211.1 mm, vias 0 -> 2
- net row0: track 0.00 -> 197.7 mm
- net col2: track 0.00 -> 193.5 mm, vias 0 -> 1
- net col0: track 0.00 -> 181.6 mm
- net col1: track 0.00 -> 171.4 mm
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- added copper zone on B.Cu, net (none)
- added copper zone on F.Cu, net (none)
Other:
- board outline added: 237.1 x 150.5 mm
- board text added: "Designed by Kyle Chiu"
- board text added: "Right Side"
